File: hardware/ZBSmartMeter.kicad_pcb (KiCad board)
At the start: 2 copper layers, 43.3 x 37.6 mm, 37 parts, among them J1 RJ12, J2 Conn_01x04, J3 Conn_01x02, J5 Screw_Terminal_01x02, J6 USB_C_Receptacle_USB2.0, SW1 SW_Push, SW2 SW_Push, U1 NCN5150DG, U2 TLV1117-33, U3 ESP32-C6-MINI-1/U

Commit message: update hardware + documentation
Other:
- board text added: "Reset"
- board text added: "ZigBee"
Changed lines of the file:
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@@
     (property "ki_keywords" "mounting hole")
     (attr exclude_from_pos_files)
-    (fp_text reference "H1" (at 0 -3.2) (layer "F.SilkS")
+    (fp_text reference "H1" (at 0 -3.2) (layer "F.SilkS") hide
         (effects (font (size 1 1) (thickness 0.15)))
     )
@@
   (gr_rect (start 161.671 83.058) (end 204.978 120.65)
     (stroke (width 0.1) (type default)) (fill none) (layer "Edge.Cuts"))
+  (gr_text "Reset" (at 162.4838 86.6394 -90) (layer "F.SilkS")
+    (effects (font (size 1 1) (thickness 0.15)) (justify left bottom))
+  )
+  (gr_text "ZigBee" (at 162.4584 112.8268 -90) (layer "F.SilkS")
+    (effects (font (size 1 1) (thickness 0.15)) (justify left bottom))
+  )
   (segment (start 184.549954 89.303702) (end 185.669954 89.303702) (width 0.25) (layer "F.Cu") (net 1))
   (segment (start 182.372 118.888296) (end 182.752266 119.268562) (width 0.5) (layer "F.Cu") (net 1))
