File: hardware/ZBSmartMeter.kicad_pcb (KiCad board)
At the start: 2 copper layers, 43.3 x 37.6 mm, 37 parts, among them J1 RJ12, J2 Conn_01x04, J3 Conn_01x02, J5 Screw_Terminal_01x02, J6 USB_C_Receptacle_USB2.0, SW1 SW_Push, SW2 SW_Push, U1 NCN5150DG, U2 TLV1117-33, U3 ESP32-C6-MINI-1/U

Commit message: LED to bright, change resistor value
Parts:
- D2: value LED/20mA -> LEDmA
- R7: value 160Ω -> 680Ω
Changed lines of the file:
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@@
         (effects (font (size 1 1) (thickness 0.15)))
     )
-    (fp_text value "160Ω" (at 0 1.43 90) (layer "F.Fab")
+    (fp_text value "680Ω" (at 0 1.43 90) (layer "F.Fab")
         (effects (font (size 1 1) (thickness 0.15)))
     )
@@
         (effects (font (size 1 1) (thickness 0.15)))
     )
-    (fp_text value "LED/20mA" (at 0 1.43 90) (layer "F.Fab")
-        (effects (font (size 1 1) (thickness 0.15)))
-    )
+    (fp_text value "LEDmA" (at 0 1.43 90) (layer "F.Fab")
+        (effects (font (size 1 1) (thickness 0.15)))
+    )

Commit message: dlms in progress
Connections:
- net UART1_PROG_RX renamed UART0_PROG_RX
Changed lines of the file:
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@@
   (net 30 "ZB_LED")
   (net 31 "UART0_PROG_TX")
-  (net 32 "UART1_PROG_RX")
+  (net 32 "UART0_PROG_RX")
   (net 33 "ZB_BUTTON")
   (net 34 "unconnected-(U1-VB-Pad2)")
@@
       (net 20 "Net-(J2-Pin_3)") (pintype "passive"))
     (pad "2" smd roundrect (at 0.825 0 180) (size 0.8 0.95) (layers "F.Cu" "F.Paste" "F.Mask") (roundrect_rratio 0.25)
-      (net 32 "UART1_PROG_RX") (pintype "passive"))
+      (net 32 "UART0_PROG_RX") (pintype "passive"))
     (model "${KICAD6_3DMODEL_DIR}/Resistor_SMD.3dshapes/R_0603_1608Metric.wrl"
       (offset (xyz 0 0 0))
@@
       (net 39 "UART1_TX") (pinfunction "GPIO23") (pintype "bidirectional"))
     (pad "30" smd rect (at 5.9 2.7 90) (size 0.4 0.8) (layers "F.Cu" "F.Paste" "F.Mask")
-      (net 32 "UART1_PROG_RX") (pinfunction "U0RXD/GPIO17") (pintype "bidirectional"))
+      (net 32 "UART0_PROG_RX") (pinfunction "U0RXD/GPIO17") (pintype "bidirectional"))
     (pad "31" smd rect (at 5.9 1.9 90) (size 0.4 0.8) (layers "F.Cu" "F.Paste" "F.Mask")
       (net 31 "UART0_PROG_TX") (pinfunction "U0TXD/GPIO16") (pintype "bidirectional"))
@@
     )
   )
-  (zone (net 32) (net_name "UART1_PROG_RX") (layer "F.Cu") (name "$teardrop_padvia$") (hatch edge 0.5)
+  (zone (net 32) (net_name "UART0_PROG_RX") (layer "F.Cu") (name "$teardrop_padvia$") (hatch edge 0.5)
     (priority 30061)
     (attr (teardrop (type padvia)))
@@
     )
   )
-  (zone (net 32) (net_name "UART1_PROG_RX") (layer "F.Cu") (name "$teardrop_padvia$") (hatch edge 0.5)
+  (zone (net 32) (net_name "UART0_PROG_RX") (layer "F.Cu") (name "$teardrop_padvia$") (hatch edge 0.5)
     (priority 30087)
     (attr (teardrop (type padvia)))
